File: KiCAD/POWER.sch (KiCad schematic (older format))
At the start: 10 parts, among them J35 Conn_01x02, J36 Conn_01x02, T1 750315371, T1_1 750315371, U12 SN6505B

Commit message: Add files via upload
Connections:
- wire segments 33 -> 25
Other:
- moved on the sheet: T1_1
Changed lines of the file:
@@
 L da2303:da2303 T1_1
 U 1 1 5CDCD766
-P 4300 4500
-F 0 "T1_1" H 4300 5215 50  0000 C CNN
-F 1 "750315371" H 4300 5124 50  0000 C CNN
-F 2 "750315371:750315371" H 4300 5033 50  0000 C CNN
-F 3 "" H 4300 4500 50  0000 C CNN
-F 4 "750315371" H 4300 4500 50  0001 C CNN "MNP"
-	1    4300 4500
+P 4200 7000
+F 0 "T1_1" H 4200 7715 50  0000 C CNN
+F 1 "750315371" H 4200 7624 50  0000 C CNN
+F 2 "750315371:750315371" H 4200 7533 50  0000 C CNN
+F 3 "" H 4200 7000 50  0000 C CNN
+F 4 "750315371" H 4200 7000 50  0001 C CNN "MNP"
+	1    4200 7000
 	1    0    0    -1
 $EndComp
@@
 2_VCC
 Wire Wire Line
-	3650 3250 3550 3250
-Wire Wire Line
 	3550 3150 3550 2850
 Wire Wire Line
@@
 	3550 3650 4200 3450
 Wire Wire Line
-	3650 3250 3650 3150
-Wire Wire Line
-	3650 3150 4000 3150
-Wire Wire Line
-	3650 3250 3650 3350
-Wire Wire Line
-	3650 3350 4200 3250
-Connection ~ 3650 3250
-Wire Wire Line
 	4600 3050 4950 2850
 Wire Wire Line
 	4600 3450 4950 3650
-Wire Wire Line
-	4800 3150 4900 3150
-Wire Wire Line
-	4900 3150 4900 3250
-Wire Wire Line
-	4900 3350 4600 3250
 Text HLabel 5700 3250 2    50   Input ~ 0
 3_OUT1A2B_DIODES
 Text HLabel 5000 3250 2    50   Input ~ 0
 4_OUT1B2A
-Wire Wire Line
-	4900 3250 5000 3250
-Connection ~ 4900 3250
-Wire Wire Line
-	4900 3250 4900 3350
 Wire Wire Line
 	5650 3250 5700 3250
@@
 	1    0    0    -1
 $EndComp
+Wire Wire Line
+	5000 3250 4600 3250
+Wire Wire Line
+	3550 3250 4200 3250
 $EndSCHEMATC
