File: KiCAD/FreeEEG32-beta.kicad_pcb (KiCad board)
At the start: 4 copper layers, 70 x 70 mm, 198 parts, among them J37 USB_B_Micro, J51 USB_B_Micro, J53 Conn_02x10_Odd_Even, J54 Conn_02x10_Odd_Even, J55 Conn_02x10_Odd_Even, J56 Conn_02x10_Odd_Even, J57 Conn_02x03_Odd_Even, J58 Conn_02x03_Odd_Even, J61 Conn_01x02, J62 Conn_01x02, J63 Conn_01x02, J64 Conn_01x02, J65 Conn_01x02, J69 Conn_01x02, J73 Conn_01x02, J78 Conn_01x02, J79 Conn_01x02, J80 Conn_01x02, J81 Conn_01x02, J82 Conn_02x02_Odd_Even, J83 Conn_02x02_Odd_Even, J85 Conn_01x02, J88 Conn_01x02, J89 Conn_01x02, J90 Conn_01x02, SW1 SW_Push, SW2 SW_Push, T1 750315371, U1 AD7779, U10 LP5907, U11 LSM6DS3, U12 SN6505B, U13 473521001, U17 ADuM3160, U18 ADUM1402BRWZ, U19 ISO7341c, U2 AD7779, U3 AD7779, U4 AD7779, U5 LP5907, U6 LP5907, U7 ADR4525, U8 FXO-SM7_OSC-SMD7050_short, U9 STM32H743ZITx, Y1 32768Hz, Y2 16MHz

Commit message: Add files via upload
Parts:
- D1, D2: footprint SOD-123:SOD−123 -> Diode_SMD:D_SOD-123
